File: kicad/vector/pic32mx_4.kicad_sch (KiCad schematic)
At the start: 7 parts, among them U9 PIC32MX695F512L-80I-PT_UNIT

Commit message: add pics & update kicad files
Parts:
- RA_5: value 1K -> 390
